File: pcb/LoRaWan_Bridge/LoRaWan_Bridge.kicad_sch (KiCad schematic)
At the start: 3 parts, among them J1 Conn_01x13, J2 Conn_01x13, J3 Conn_02x04_Odd_Even

Commit message: PCB updates to fix pin spacing
Parts:
- added BT2: BK-18650-PC2, BAT_BK-18650-PC2, symbol BK-18650-PC2:BK-18650-PC2
Connections:
- net GND: now also BT2.-
- new net +BATT: BT2.+
Changed lines of the file:
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@@
+    (stroke (width 0) (type default))
+  )
+  (wire (pts (xy 162.56 54.61) (xy 162.56 58.42))
+    (stroke (width 0) (type default))
+  )
+  (wire (pts (xy 181.61 58.42) (xy 181.61 62.23))
     (stroke (width 0) (type default))
   )
@@
   )
   (wire (pts (xy 125.73 55.88) (xy 121.92 55.88))
+    (stroke (width 0) (type default))
+  )
+  (wire (pts (xy 162.56 58.42) (xy 166.37 58.42))
     (stroke (width 0) (type default))
   )
@@
     )
   )
+  (symbol (lib_id "BK-18650-PC2:BK-18650-PC2") (at 173.99 58.42 0) (unit 1)
+    (in_bom yes) (on_board yes) (dnp no) (fields_autoplaced)
+    (property "Reference" "BT2" (at 173.355 52.07 0)
+      (effects (font (size 1.27 1.27)))
+    )
+    (property "Value" "BK-18650-PC2" (at 173.355 54.61 0)
+      (effects (font (size 1.27 1.27)))
+    )
+    (property "Footprint" "BAT_BK-18650-PC2" (at 173.99 58.42 0)
+      (effects (font (size 1.27 1.27)) (justify bottom) hide)
+    )
+    (property "Datasheet" "" (at 173.99 58.42 0)
+      (effects (font (size 1.27 1.27)) hide)
+    )
+    (property "PARTREV" "F" (at 173.99 58.42 0)
+      (effects (font (size 1.27 1.27)) (justify bottom) hide)
+    )
+    (property "STANDARD" "Manufacturer Recommendations" (at 173.99 58.42 0)
+      (effects (font (size 1.27 1.27)) (justify bottom) hide)
+    )
+    (property "MAXIMUM_PACKAGE_HEIGHT" "21.41 mm" (at 173.99 58.42 0)
+      (effects (font (size 1.27 1.27)) (justify bottom) hide)
+    )
+    (property "MANUFACTURER" "MPD" (at 173.99 58.42 0)
+      (effects (font (size 1.27 1.27)) (justify bottom) hide)
+    )
+    (pin "+")
+    (pin "-")
+    (instances
+      (project "LoRaWan_Bridge"
+        (path "/17b7df2a-59af-47ab-8a19-d72902de2b41"
+          (reference "BT2") (unit 1)
+        )
+      )
+    )
+  )
+  (symbol (lib_id "power:+BATT") (at 162.56 54.61 0) (unit 1)
+    (in_bom yes) (on_board yes) (dnp no) (fields_autoplaced)
+    (property "Reference" "#PWR05" (at 162.56 58.42 0)
+      (effects (font (size 1.27 1.27)) hide)
+    )
+    (property "Value" "+BATT" (at 162.56 50.8 0)
+      (effects (font (size 1.27 1.27)))
+    )
+    (property "Footprint" "" (at 162.56 54.61 0)
+      (effects (font (size 1.27 1.27)) hide)
+    )
+    (property "Datasheet" "" (at 162.56 54.61 0)
+      (effects (font (size 1.27 1.27)) hide)
+    )
+    (pin "1")
+    (instances
+      (project "LoRaWan_Bridge"
+        (path "/17b7df2a-59af-47ab-8a19-d72902de2b41"
+          (reference "#PWR05") (unit 1)
+        )
+      )
+    )
+  )
   (symbol (lib_id "power:GND") (at 77.47 60.96 0) (unit 1)
     (in_bom yes) (on_board yes) (dnp no) (fields_autoplaced)
@@
         )
       )
+    )
+  )
+  (symbol (lib_id "power:GND") (at 181.61 62.23 0) (unit 1)
+    (in_bom yes) (on_board yes) (dnp no) (fields_autoplaced)
+    (property "Reference" "#PWR06" (at 181.61 68.58 0)
+      (effects (font (size 1.27 1.27)) hide)
+    )
+    (property "Value" "GND" (at 181.61 67.31 0)
+      (effects (font (size 1.27 1.27)))
+    )
+    (property "Footprint" "" (at 181.61 62.23 0)
+      (effects (font (size 1.27 1.27)) hide)
+    )
+    (property "Datasheet" "" (at 181.61 62.23 0)
+      (effects (font (size 1.27 1.27)) hide)
+    )
+    (pin "1")
+    (instances
+      (project "LoRaWan_Bridge"
+        (path "/17b7df2a-59af-47ab-8a19-d72902de2b41"
+          (reference "#PWR06") (unit 1)
+        )
+      )
